File: 2x2-MacroPad/2x2-MacroPad.kicad_sch (KiCad schematic)
At the start: 9 parts, among them U1 ATmega32U4-A

Commit message: ""
Parts:
- removed C4: C_Small, symbol Device:C_Small
- added C6: 0.1uF, symbol Device:C_Small
- C2, C5: value C_Small -> 0.1uF
- C3: value C_Small -> 10uF
Connections:
- net +5V: now also C2.1, C3.1, C5.1, U1.7 (VBUS), C6.1
- net GND: now also C2.2, C3.2, C5.2, C6.2
Other:
- moved on the sheet: C5
Changed lines of the file:
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@@
   (junction (at 132.08 132.08) (diameter 0) (color 0 0 0 0)
   )
+  (junction (at 78.74 106.68) (diameter 0) (color 0 0 0 0)
+  )
   (junction (at 134.62 40.64) (diameter 0) (color 0 0 0 0)
   )
+  (junction (at 73.66 113.03) (diameter 0) (color 0 0 0 0)
+  )
+  (junction (at 78.74 113.03) (diameter 0) (color 0 0 0 0)
+  )
   (junction (at 132.08 40.64) (diameter 0) (color 0 0 0 0)
   )
+  (junction (at 73.66 106.68) (diameter 0) (color 0 0 0 0)
+  )
+  (junction (at 68.58 113.03) (diameter 0) (color 0 0 0 0)
+  )
+  (junction (at 68.58 106.68) (diameter 0) (color 0 0 0 0)
+  )
   (wire (pts (xy 134.62 40.64) (xy 132.08 40.64))
     (stroke (width 0) (type default))
   )
+  (wire (pts (xy 68.58 111.76) (xy 68.58 113.03))
+    (stroke (width 0) (type default))
+  )
   (wire (pts (xy 81.28 73.66) (xy 102.87 73.66))
     (stroke (width 0) (type default))
   )
+  (wire (pts (xy 58.42 113.03) (xy 58.42 111.76))
+    (stroke (width 0) (type default))
+  )
+  (wire (pts (xy 78.74 106.68) (xy 88.9 106.68))
+    (stroke (width 0) (type default))
+  )
+  (wire (pts (xy 111.76 68.58) (xy 119.38 68.58))
+    (stroke (width 0) (type default))
+  )
   (wire (pts (xy 106.68 81.28) (xy 106.68 83.82))
     (stroke (width 0) (type default))
@@
     (stroke (width 0) (type default))
   )
+  (wire (pts (xy 88.9 111.76) (xy 88.9 113.03))
+    (stroke (width 0) (type default))
+  )
   (wire (pts (xy 107.95 73.66) (xy 119.38 73.66))
     (stroke (width 0) (type default))
   )
+  (wire (pts (xy 73.66 113.03) (xy 78.74 113.03))
+    (stroke (width 0) (type default))
+  )
   (wire (pts (xy 132.08 132.08) (xy 134.62 132.08))
     (stroke (width 0) (type default))
   )
+  (wire (pts (xy 73.66 101.6) (xy 73.66 106.68))
+    (stroke (width 0) (type default))
+  )
+  (wire (pts (xy 73.66 113.03) (xy 73.66 115.57))
+    (stroke (width 0) (type default))
+  )
   (wire (pts (xy 134.62 40.64) (xy 137.16 40.64))
     (stroke (width 0) (type default))
@@
     (stroke (width 0) (type default))
   )
+  (wire (pts (xy 58.42 106.68) (xy 68.58 106.68))
+    (stroke (width 0) (type default))
+  )
+  (wire (pts (xy 88.9 113.03) (xy 78.74 113.03))
+    (stroke (width 0) (type default))
+  )
+  (wire (pts (xy 68.58 113.03) (xy 58.42 113.03))
+    (stroke (width 0) (type default))
+  )
+  (wire (pts (xy 111.76 67.31) (xy 111.76 68.58))
+    (stroke (width 0) (type default))
+  )
+  (wire (pts (xy 68.58 113.03) (xy 73.66 113.03))
+    (stroke (width 0) (type default))
+  )
   (wire (pts (xy 121.92 134.62) (xy 132.08 134.62))
     (stroke (width 0) (type default))
   )
+  (wire (pts (xy 73.66 106.68) (xy 78.74 106.68))
+    (stroke (width 0) (type default))
+  )
   (wire (pts (xy 162.56 101.6) (xy 172.72 101.6))
     (stroke (width 0) (type default))
@@
     (stroke (width 0) (type default))
   )
-  (symbol (lib_id "Device:C_Small") (at 95.25 109.22 0) (unit 1)
-    (in_bom yes) (on_board yes) (dnp no) (fields_autoplaced)
-    (property "Reference" "C4" (at 97.79 108.5913 0)
-      (effects (font (size 1.27 1.27)) (justify left))
-    )
-    (property "Value" "C_Small" (at 97.79 111.1313 0)
-      (effects (font (size 1.27 1.27)) (justify left))
-    )
-    (property "Footprint" "" (at 95.25 109.22 0)
-      (effects (font (size 1.27 1.27)) hide)
-    )
-    (property "Datasheet" "~" (at 95.25 109.22 0)
-      (effects (font (size 1.27 1.27)) hide)
-    )
-    (pin "1")
-    (pin "2")
-    (instances
-      (project "2x2-MacroPad"
-        (path "/511aa040-d6a3-4810-aeed-27ccce4f72f8"
-          (reference "C4") (unit 1)
+  (wire (pts (xy 78.74 113.03) (xy 78.74 111.76))
+    (stroke (width 0) (type default))
+  )
+  (wire (pts (xy 68.58 106.68) (xy 73.66 106.68))
+    (stroke (width 0) (type default))
+  )
+  (symbol (lib_id "power:+5V") (at 73.66 101.6 0) (unit 1)
+    (in_bom yes) (on_board yes) (dnp no) (fields_autoplaced)
+    (property "Reference" "#PWR05" (at 73.66 105.41 0)
+      (effects (font (size 1.27 1.27)) hide)
+    )
+    (property "Value" "+5V" (at 73.66 97.79 0)
+      (effects (font (size 1.27 1.27)))
+    )
+    (property "Footprint" "" (at 73.66 101.6 0)
+      (effects (font (size 1.27 1.27)) hide)
+    )
+    (property "Datasheet" "" (at 73.66 101.6 0)
+      (effects (font (size 1.27 1.27)) hide)
+    )
+    (pin "1")
+    (instances
+      (project "2x2-MacroPad"
+        (path "/511aa040-d6a3-4810-aeed-27ccce4f72f8"
+          (reference "#PWR05") (unit 1)
         )
       )
@@
       (effects (font (size 1.27 1.27)) (justify left))
     )
-    (property "Value" "C_Small" (at 71.12 111.1313 0)
+    (property "Value" "0.1uF" (at 71.12 111.1313 0)
       (effects (font (size 1.27 1.27)) (justify left))
     )
@@
     )
   )
-  (symbol (lib_id "Device:C_Small") (at 82.55 109.22 0) (unit 1)
-    (in_bom yes) (on_board yes) (dnp no) (fields_autoplaced)
-    (property "Reference" "C3" (at 85.09 108.5913 0)
-      (effects (font (size 1.27 1.27)) (justify left))
-    )
-    (property "Value" "C_Small" (at 85.09 111.1313 0)
-      (effects (font (size 1.27 1.27)) (justify left))
-    )
-    (property "Footprint" "" (at 82.55 109.22 0)
-      (effects (font (size 1.27 1.27)) hide)
-    )
-    (property "Datasheet" "~" (at 82.55 109.22 0)
+  (symbol (lib_id "Device:C_Small") (at 88.9 109.22 0) (unit 1)
+    (in_bom yes) (on_board yes) (dnp no) (fields_autoplaced)
+    (property "Reference" "C3" (at 91.44 108.5913 0)
+      (effects (font (size 1.27 1.27)) (justify left))
+    )
+    (property "Value" "10uF" (at 91.44 111.1313 0)
+      (effects (font (size 1.27 1.27)) (justify left))
+    )
+    (property "Footprint" "" (at 88.9 109.22 0)
+      (effects (font (size 1.27 1.27)) hide)
+    )
+    (property "Datasheet" "~" (at 88.9 109.22 0)
       (effects (font (size 1.27 1.27)) hide)
     )
@@
     )
   )
+  (symbol (lib_id "power:+5V") (at 111.76 67.31 0) (unit 1)
+    (in_bom yes) (on_board yes) (dnp no) (fields_autoplaced)
+    (property "Reference" "#PWR07" (at 111.76 71.12 0)
+      (effects (font (size 1.27 1.27)) hide)
+    )
+    (property "Value" "+5V" (at 111.76 63.5 0)
+      (effects (font (size 1.27 1.27)))
+    )
+    (property "Footprint" "" (at 111.76 67.31 0)
+      (effects (font (size 1.27 1.27)) hide)
+    )
+    (property "Datasheet" "" (at 111.76 67.31 0)
+      (effects (font (size 1.27 1.27)) hide)
+    )
+    (pin "1")
+    (instances
+      (project "2x2-MacroPad"
+        (path "/511aa040-d6a3-4810-aeed-27ccce4f72f8"
+          (reference "#PWR07") (unit 1)
+        )
+      )
+    )
+  )
   (symbol (lib_id "Device:R_Small") (at 105.41 73.66 90) (unit 1)
     (in_bom yes) (on_board yes) (dnp no) (fields_autoplaced)
@@
     )
   )
-  (symbol (lib_id "Device:C_Small") (at 59.69 109.22 0) (unit 1)
-    (in_bom yes) (on_board yes) (dnp no) (fields_autoplaced)
-    (property "Reference" "C5" (at 62.23 108.5913 0)
-      (effects (font (size 1.27 1.27)) (justify left))
-    )
-    (property "Value" "C_Small" (at 62.23 111.1313 0)
-      (effects (font (size 1.27 1.27)) (justify left))
-    )
-    (property "Footprint" "" (at 59.69 109.22 0)
-      (effects (font (size 1.27 1.27)) hide)
-    )
-    (property "Datasheet" "~" (at 59.69 109.22 0)
+  (symbol (lib_id "Device:C_Small") (at 58.42 109.22 0) (unit 1)
+    (in_bom yes) (on_board yes) (dnp no) (fields_autoplaced)
+    (property "Reference" "C5" (at 60.96 108.5913 0)
+      (effects (font (size 1.27 1.27)) (justify left))
+    )
+    (property "Value" "0.1uF" (at 60.96 111.1313 0)
+      (effects (font (size 1.27 1.27)) (justify left))
+    )
+    (property "Footprint" "" (at 58.42 109.22 0)
+      (effects (font (size 1.27 1.27)) hide)
+    )
+    (property "Datasheet" "~" (at 58.42 109.22 0)
       (effects (font (size 1.27 1.27)) hide)
     )
@@
         (path "/511aa040-d6a3-4810-aeed-27ccce4f72f8"
           (reference "C5") (unit 1)
+        )
+      )
+    )
+  )
+  (symbol (lib_id "Device:C_Small") (at 78.74 109.22 0) (unit 1)
+    (in_bom yes) (on_board yes) (dnp no) (fields_autoplaced)
+    (property "Reference" "C6" (at 81.28 108.5913 0)
+      (effects (font (size 1.27 1.27)) (justify left))
+    )
+    (property "Value" "0.1uF" (at 81.28 111.1313 0)
+      (effects (font (size 1.27 1.27)) (justify left))
+    )
+    (property "Footprint" "" (at 78.74 109.22 0)
+      (effects (font (size 1.27 1.27)) hide)
+    )
+    (property "Datasheet" "~" (at 78.74 109.22 0)
+      (effects (font (size 1.27 1.27)) hide)
+    )
+    (pin "1")
+    (pin "2")
+    (instances
+      (project "2x2-MacroPad"
+        (path "/511aa040-d6a3-4810-aeed-27ccce4f72f8"
+          (reference "C6") (unit 1)
         )
       )
@@
         )
       )
+    )
+  )
+  (symbol (lib_id "power:GND") (at 73.66 115.57 0) (unit 1)
+    (in_bom yes) (on_board yes) (dnp no) (fields_autoplaced)
+    (property "Reference" "#PWR06" (at 73.66 121.92 0)
+      (effects (font (size 1.27 1.27)) hide)
+    )
+    (property "Value" "GND" (at 73.66 120.65 0)
+      (effects (font (size 1.27 1.27)))
+    )
+    (property "Footprint" "" (at 73.66 115.57 0)
+      (effects (font (size 1.27 1.27)) hide)
+    )
+    (property "Datasheet" "" (at 73.66 115.57 0)
+      (effects (font (size 1.27 1.27)) hide)
+    )
+    (pin "1")
+    (instances
+      (project "2x2-MacroPad"
+        (path "/511aa040-d6a3-4810-aeed-27ccce4f72f8"
+          (reference "#PWR06") (unit 1)
+        )
+      )

Commit message: Finished Schematic
Parts:
- added C4, C7: 22pF, Capacitor_SMD:C_0805_2012Metric, symbol Device:C_Small
- added D1, D2, D3, D4: SOD-123, Diode_SMD:D_SOD-123, symbol Device:D_Small
- added F1: 500mA, Fuse:Fuse_1206_3216Metric, symbol Device:Polyfuse_Small
- added MX1, MX2, MX3, MX4: MX-NoLED, MX_Alps_Hybrid:MX-1U-NoLED, symbol MX_Alps_Hybrid:MX-NoLED
- added R4: 10k, Resistor_SMD:R_0805_2012Metric, symbol Device:R_Small
- added SW1: SW_Push, random-keyboard-parts:SKQG-1155865, symbol Switch:SW_Push
- added USB1: Molex-0548190589, random-keyboard-parts:Molex-0548190589, symbol random-keyboard-parts:Molex-0548190589
- added Y1: 16MHz, Package_QFP:TQFP-44_10x10mm_P0.8mm, symbol Device:Crystal_GND24_Small
- C1, C2, C3, C5, C6: footprint (none) -> Capacitor_SMD:C_0805_2012Metric
- R1: footprint (none) -> Resistor_SMD:R_0805_2012Metric
- R2, R3: value R_Small -> 22; footprint (none) -> Resistor_SMD:R_0805_2012Metric
Connections:
- net +5V: now also F1.2, R4.1
- net GND: now also C4.1, C7.1, SW1.1, USB1.1 (GND), USB1.6 (SHIELD), Y1.2, Y1.4
- net at U1.13 (~{RESET}): now also R4.2, SW1.2
- net at U1.16 (XTAL2): now also C7.2, Y1.3
- net at U1.17 (XTAL1): now also C4.2, Y1.1
- net D-: now reaches R3.1
- net D-: now also USB1.3 (D+)
- net D+: now reaches R2.1
- net D+: now also USB1.4 (D-)
- new net: D1.2 (A), MX1.2 (ROW)
- new net: D3.2 (A), MX3.2 (ROW)
- new net: D4.2 (A), MX4.2 (ROW)
- new net: D2.2 (A), MX2.2 (ROW)
- new net COL0: MX1.1 (COL), MX3.1 (COL)
- new net COL1: MX2.1 (COL), MX4.1 (COL)
- new net ROW0: D1.1 (K), D2.1 (K)
- new net ROW1: D3.1 (K), D4.1 (K)
- new net VCC: F1.1, USB1.5 (VBUS)

Commit message: Started PCB routing
Parts:
- Y1: footprint Package_QFP:TQFP-44_10x10mm_P0.8mm -> Crystal:Crystal_SMD_3225-4Pin_3.2x2.5mm_HandSoldering
Changed lines of the file:
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@@
       (effects (font (size 1.27 1.27)))
     )
-    (property "Footprint" "Package_QFP:TQFP-44_10x10mm_P0.8mm" (at 106.68 55.88 0)
+    (property "Footprint" "Crystal:Crystal_SMD_3225-4Pin_3.2x2.5mm_HandSoldering" (at 106.68 55.88 0)
       (effects (font (size 1.27 1.27)) hide)
     )
