File: 2x2-MacroPad/2x2-MacroPad.kicad_sch (KiCad schematic)
At the start: 24 parts, among them SW1 SW_Push, U1 ATmega32U4-A, Y1 16MHz

Commit message: Finished Routing
Connections:
- net COL0: now also U1.29 (PB5)
- net COL1: now also U1.28 (PB4)
- net ROW0: now also U1.27 (PD7)
- net ROW1: now also U1.30 (PB6)
Changed lines of the file:
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@@
+    (stroke (width 0) (type default))
+  )
+  (wire (pts (xy 154.94 93.98) (xy 158.75 93.98))
     (stroke (width 0) (type default))
   )
@@
     (stroke (width 0) (type default))
   )
+  (wire (pts (xy 156.21 57.15) (xy 156.845 57.15))
+    (stroke (width 0) (type default))
+  )
   (wire (pts (xy 109.22 55.88) (xy 109.22 63.5))
     (stroke (width 0) (type default))
@@
     (stroke (width 0) (type default))
   )
+  (wire (pts (xy 154.94 96.52) (xy 154.94 93.98))
+    (stroke (width 0) (type default))
+  )
   (wire (pts (xy 204.47 78.74) (xy 208.28 78.74))
     (stroke (width 0) (type default))
@@
     (stroke (width 0) (type default))
   )
+  (wire (pts (xy 156.21 58.42) (xy 149.86 58.42))
+    (stroke (width 0) (type default))
+  )
+  (wire (pts (xy 156.21 63.5) (xy 149.86 63.5))
+    (stroke (width 0) (type default))
+  )
+  (wire (pts (xy 149.86 96.52) (xy 154.94 96.52))
+    (stroke (width 0) (type default))
+  )
   (wire (pts (xy 194.31 83.82) (xy 204.47 83.82))
     (stroke (width 0) (type default))
@@
     (stroke (width 0) (type default))
   )
+  (wire (pts (xy 149.86 60.96) (xy 156.845 60.96))
+    (stroke (width 0) (type default))
+  )
   (wire (pts (xy 132.08 35.56) (xy 132.08 40.64))
     (stroke (width 0) (type default))
@@
     (stroke (width 0) (type default))
   )
+  (wire (pts (xy 156.21 57.15) (xy 156.21 58.42))
+    (stroke (width 0) (type default))
+  )
   (wire (pts (xy 194.31 101.6) (xy 204.47 101.6))
     (stroke (width 0) (type default))
@@
     (stroke (width 0) (type default))
   )
+  (wire (pts (xy 156.21 64.77) (xy 156.21 63.5))
+    (stroke (width 0) (type default))
+  )
   (wire (pts (xy 229.87 45.72) (xy 232.41 45.72))
     (stroke (width 0) (type default))
@@
   )
   (wire (pts (xy 162.56 101.6) (xy 172.72 101.6))
+    (stroke (width 0) (type default))
+  )
+  (wire (pts (xy 156.21 64.77) (xy 156.845 64.77))
     (stroke (width 0) (type default))
   )
@@
     )
   )
+  (global_label "COL1" (shape input) (at 156.845 57.15 0) (fields_autoplaced)
+    (effects (font (size 1.27 1.27)) (justify left))
+    (property "Intersheetrefs" "${INTERSHEET_REFS}" (at 164.5889 57.15 0)
+      (effects (font (size 1.27 1.27)) (justify left) hide)
+    )
+  )
   (global_label "D+" (shape input) (at 81.28 72.39 180) (fields_autoplaced)
     (effects (font (size 1.27 1.27)) (justify right))
@@
     )
   )
+  (global_label "ROW0" (shape input) (at 158.75 93.98 0) (fields_autoplaced)
+    (effects (font (size 1.27 1.27)) (justify left))
+    (property "Intersheetrefs" "${INTERSHEET_REFS}" (at 166.9172 93.98 0)
+      (effects (font (size 1.27 1.27)) (justify left) hide)
+    )
+  )
   (global_label "COL0" (shape input) (at 213.36 64.77 90) (fields_autoplaced)
     (effects (font (size 1.27 1.27)) (justify left))
@@
     )
   )
+  (global_label "ROW1" (shape input) (at 156.845 64.77 0) (fields_autoplaced)
+    (effects (font (size 1.27 1.27)) (justify left))
+    (property "Intersheetrefs" "${INTERSHEET_REFS}" (at 165.0122 64.77 0)
+      (effects (font (size 1.27 1.27)) (justify left) hide)
+    )
+  )
+  (global_label "COL0" (shape input) (at 156.845 60.96 0) (fields_autoplaced)
+    (effects (font (size 1.27 1.27)) (justify left))
+    (property "Intersheetrefs" "${INTERSHEET_REFS}" (at 164.5889 60.96 0)
+      (effects (font (size 1.27 1.27)) (justify left) hide)
+    )
+  )
